File: hardware/electrical/buck-converter/KiCAD/schaltung.kicad_pcb (KiCad board)
At the start: 2 copper layers, 89 x 50 mm, 23 parts, among them J1 V_in +, J10 GND, J2 V_in -, J3 V_OUT +, J4 V_OUT -, J5 PWM +, J6 I +, J7 U +, J8 GND, J9 GND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

Commit message: Updated PCBs; added Bleed Resistor and fixed Frontend GND connections
Parts:
- removed J9: GND, MountingHole:MountingHole_2.2mm_M2_Pad
- added R4_Bleed1: 100k, Resistor_SMD:R_1206_3216Metric, F.Cu at (143.5, 63.5)
- C1: value 470µF -> 1000µF
- C2: value C -> 1µF
- moved C1 7.00 mm to (127.0, 56.5)
- moved C2 5.07 mm to (138.4, 56.5)
- moved L1 2.77 mm to (114.3, 55.9)
Routing:
- net Net-(J3-Pin_1): track 46.2 -> 54.7 mm
- net Net-(D1-K): track 22.4 -> 19.1 mm
Changed lines of the file:
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@@
 	(footprint "Resistor_SMD:R_1206_3216Metric"
 		(layer "F.Cu")
+		(at 143.51 63.5 -90)
+		(descr "Resistor SMD 1206 (3216 Metric), square (rectangular) end terminal, IPC-7351 nominal, (Body size source: IPC-SM-782 page 72, https://www.pcb-3d.com/wordpress/wp-content/uploads/ipc-sm-782a_amendment_1_and_2.pdf), generated with kicad-footprint-generator")
+		(tags "resistor")
+		(property "Reference" "R4_Bleed1"
+			(at 0 -1.83 90)
+			(layer "F.SilkS")
+			(effects
+				(font
+					(size 1 1)
+					(thickness 0.15)
+				)
+			)
+		)
+		(property "Value" "100k"
+			(at 0 1.83 90)
+			(layer "F.Fab")
+			(effects
+				(font
+					(size 1 1)
+					(thickness 0.15)
+				)
+			)
+		)
+		(property "Datasheet" ""
+			(at 0 0 90)
+			(layer "F.Fab")
+			(hide yes)
+			(effects
+				(font
+					(size 1.27 1.27)
+					(thickness 0.15)
+				)
+			)
+		)
+		(property "Description" "Resistor"
+			(at 0 0 90)
+			(layer "F.Fab")
+			(hide yes)
+			(effects
+				(font
+					(size 1.27 1.27)
+					(thickness 0.15)
+				)
+			)
+		)
+		(property ki_fp_filters "R_*")
+		(sheetname "/")
+		(sheetfile "schaltung.kicad_sch")
+		(attr smd)
+		(fp_line
+			(start -0.727064 0.91)
+			(end 0.727064 0.91)
+			(stroke
+				(width 0.12)
+				(type solid)
+			)
+			(layer "F.SilkS")
+		)
+		(fp_line
+			(start -0.727064 -0.91)
+			(end 0.727064 -0.91)
+			(stroke
+				(width 0.12)
+				(type solid)
+			)
+			(layer "F.SilkS")
+		)
+		(fp_line
+			(start -2.28 1.13)
+			(end -2.28 -1.13)
+			(stroke
+				(width 0.05)
+				(type solid)
+			)
+			(layer "F.CrtYd")
+		)
+		(fp_line
+			(start 2.28 1.13)
+			(end -2.28 1.13)
+			(stroke
+				(width 0.05)
+				(type solid)
+			)
+			(layer "F.CrtYd")
+		)
+		(fp_line
+			(start -2.28 -1.13)
+			(end 2.28 -1.13)
+			(stroke
+				(width 0.05)
+				(type solid)
+			)
+			(layer "F.CrtYd")
+		)
+		(fp_line
+			(start 2.28 -1.13)
+			(end 2.28 1.13)
+			(stroke
+				(width 0.05)
+				(type solid)
+			)
+			(layer "F.CrtYd")
+		)
+		(fp_line
+			(start -1.6 0.8)
+			(end -1.6 -0.8)
+			(stroke
+				(width 0.1)
+				(type solid)
+			)
+			(layer "F.Fab")
+		)
+		(fp_line
+			(start 1.6 0.8)
+			(end -1.6 0.8)
+			(stroke
+				(width 0.1)
+				(type solid)
+			)
+			(layer "F.Fab")
+		)
+		(fp_line
+			(start -1.6 -0.8)
+			(end 1.6 -0.8)
+			(stroke
+				(width 0.1)
+				(type solid)
+			)
+			(layer "F.Fab")
+		)
+		(fp_line
+			(start 1.6 -0.8)
+			(end 1.6 0.8)
+			(stroke
+				(width 0.1)
+				(type solid)
+			)
+			(layer "F.Fab")
+		)
+		(fp_text user "${REFERENCE}"
+			(at 0 3.81 90)
+			(layer "F.Fab")
+			(effects
+				(font
+					(size 0.8 0.8)
+					(thickness 0.12)
+				)
+			)
+		)
+		(pad "1" smd roundrect
+			(at -1.4625 0 270)
+			(size 1.125 1.75)
+			(layers "F.Cu" "F.Mask" "F.Paste")
+			(roundrect_rratio 0.222222)
+			(net 2 "Net-(J3-Pin_1)")
+			(pintype "passive")
+		)
+		(pad "2" smd roundrect
+			(at 1.4625 0 270)
+			(size 1.125 1.75)
+			(layers "F.Cu" "F.Mask" "F.Paste")
+			(roundrect_rratio 0.222222)
+			(net 6 "Net-(J4-Pin_1)")
+			(pintype "passive")
+		)
+		(embedded_fonts no)
+		(model "${KICAD9_3DMODEL_DIR}/Resistor_SMD.3dshapes/R_1206_3216Metric.step"
+			(offset
+				(xyz 0 0 0)
+			)
+			(scale
+				(xyz 1 1 1)
+			)
+			(rotate
+				(xyz 0 0 0)
+			)
+		)
+	)
+	(footprint "Resistor_SMD:R_1206_3216Metric"
+		(layer "F.Cu")
 		(at 126.5 87)
 		(descr "Resistor SMD 1206 (3216 Metric), square (rectangular) end terminal, IPC-7351 nominal, (Body size source: IPC-SM-782 page 72, https://www.pcb-3d.com/wordpress/wp-content/uploads/ipc-sm-782a_amendment_1_and_2.pdf), generated with kicad-footprint-generator")
@@
 		(embedded_fonts no)
 	)
-	(footprint "MountingHole:MountingHole_2.2mm_M2_Pad"
-		(layer "F.Cu")
-		(at 85 88.5 180)
-		(descr "Mounting Hole 2.2mm, M2, generated by kicad-footprint-generator mountinghole.py")
-		(tags "mountinghole M2")
-		(property "Reference" "J9"
-			(at -0.5 -4.05 0)
-			(layer "F.SilkS")
-			(effects
-				(font
-					(size 1 1)
-					(thickness 0.15)
-				)
-			)
-		)
-		(property "Value" "GND"
-			(at 0 3.15 0)
-			(layer "F.SilkS")
-			(effects
-				(font
-					(size 1 1)
-					(thickness 0.15)
-				)
-			)
-		)
-		(property "Datasheet" ""
-			(at 0 0 0)
-			(layer "F.Fab")
-			(hide yes)
-			(effects
-				(font
-					(size 1.27 1.27)
-					(thickness 0.15)
-				)
-			)
-		)
-		(property "Description" "Generic connector, single row, 01x01, script generated"
-			(at 0 0 0)
-			(layer "F.Fab")
-			(hide yes)
-			(effects
-				(font
-					(size 1.27 1.27)
-					(thickness 0.15)
-				)
-			)
-		)
-		(property ki_fp_filters "Connector*:*_1x??_*")
-		(sheetname "/")
-		(sheetfile "schaltung.kicad_sch")
-		(attr exclude_from_pos_files)
-		(fp_circle
-			(center 0 0)
-			(end 2.2 0)
-			(stroke
-				(width 0.15)
-				(type solid)
-			)
-			(fill no)
-			(layer "Cmts.User")
-		)
-		(fp_circle
-			(center 0 0)
-			(end 2.45 0)
-			(stroke
-				(width 0.05)
-				(type solid)
-			)
-			(fill no)
-			(layer "F.CrtYd")
-		)
-		(fp_text user "${REFERENCE}"
-			(at 0 0 0)
-			(layer "F.Fab")
-			(effects
-				(font
-					(size 1 1)
-					(thickness 0.15)
-				)
-			)
-		)
-		(pad "1" thru_hole circle
-			(at 0 0 180)
-			(size 4.4 4.4)
-			(drill 2.2)
-			(layers "*.Cu" "*.Mask")
-			(remove_unused_layers no)
-			(net 1 "GND")
-			(pinfunction "Pin_1")
-			(pintype "passive")
-			(zone_connect 2)
-		)
-		(embedded_fonts no)
-	)
 	(footprint "MountingHole:MountingHole_2.2mm_M2"
 		(layer "F.Cu")
@@
 	(footprint "Capacitor_THT:C_Disc_D5.0mm_W2.5mm_P5.00mm"
 		(layer "F.Cu")
-		(at 143.5 56.5 -90)
+		(at 138.43 56.5 -90)
 		(descr "C, Disc series, Radial, pin pitch=5.00mm, diameter*width=5*2.5mm^2, Capacitor, http://cdn-reichelt.de/documents/datenblatt/B300/DS_KERKO_TC.pdf")
 		(tags "C Disc series Radial pin pitch 5.00mm diameter 5mm width 2.5mm Capacitor")
@@
 			)
 		)
-		(property "Value" "C"
+		(property "Value" "1µF"
 			(at 2.5 2.5 90)
 			(layer "F.Fab")
@@
 	(footprint "Inductor_SMD:L_Sunlord_MWSA1003S"
 		(layer "F.Cu")
-		(at 117 56.5)
+		(at 114.3 55.88)
 		(descr "Inductor, Sunlord, MWSA1003S, 11.5x10.0x2.8mm, (https://sunlordinc.com/Download.aspx?file=L1VwbG9hZEZpbGVzL1BERl9DYXQvMjAyMjExMTUxNDQ4MDU0NTQucGRm&lan=en), generated with kicad-footprint-generator gen_inductor.py")
 		(tags "Inductor mwsa")
@@
 	(footprint "Capacitor_THT:CP_Radial_D10.0mm_P5.00mm"
 		(layer "F.Cu")
-		(at 134 56.5 -90)
+		(at 127 56.5 -90)
 		(descr "CP, Radial series, Radial, pin pitch=5.00mm, diameter=10mm, height=16mm, Electrolytic Capacitor")
 		(tags "CP Radial series Radial pin pitch 5.00mm diameter 10mm height 16mm Electrolytic Capacitor")
@@
 			)
 		)
-		(property "Value" "470µF"
-			(at 2.5 6.25 90)
+		(property "Value" "1000µF"
+			(at 9.54 -1.27 180)
 			(layer "F.SilkS")
 			(effects
@@
 	)
 	(segment
+		(start 119.67 56.5)
+		(end 143.5 56.5)
+		(width 1.5)
+		(layer "F.Cu")
+		(net 2)
+	)
+	(segment
 		(start 151 63.5)
 		(end 155.5 63.5)
@@
 	)
 	(segment
-		(start 134 56.5)
-		(end 143.5 56.5)
-		(width 1.5)
+		(start 143.51 62.0375)
+		(end 143.51 56.51)
+		(width 1)
 		(layer "F.Cu")
 		(net 2)
 	)
 	(segment
-		(start 121.75 56.5)
-		(end 134 56.5)
+		(start 119.05 55.88)
+		(end 119.67 56.5)
 		(width 1.5)
 		(layer "F.Cu")
@@
 	)
 	(segment
+		(start 143.51 56.51)
+		(end 143.5 56.5)
+		(width 0.2)
+		(layer "F.Cu")
+		(net 2)
+	)
+	(segment
 		(start 144 56.5)
 		(end 151 63.5)
@@
 	)
 	(segment
-		(start 103 59)
-		(end 109.75 59)
+		(start 98.95 54.95)
+		(end 103 59)
 		(width 1.5)
 		(layer "F.Cu")
@@
 	)
 	(segment
-		(start 109.75 59)
-		(end 112.25 56.5)
+		(start 92.54 54.95)
+		(end 98.95 54.95)
 		(width 1.5)
 		(layer "F.Cu")
@@
 	)
 	(segment
-		(start 98.95 54.95)
-		(end 103 59)
+		(start 107.33 56.5)
+		(end 108.93 56.5)
 		(width 1.5)
 		(layer "F.Cu")
@@
 	)
 	(segment
-		(start 92.54 54.95)
-		(end 98.95 54.95)
+		(start 103 59)
+		(end 104.83 59)
+		(width 1.5)
+		(layer "F.Cu")
+		(net 3)
+	)
+	(segment
+		(start 104.83 59)
+		(end 107.33 56.5)
 		(width 1.5)
 		(layer "F.Cu")
